File: SBC6309BackMemory.kicad_pcb (KiCad board)
At the start: 2 copper layers, 99.4 x 102.4 mm, 11 parts, among them J3 Conn_01x16, J4 Conn_01x08, J5 Conn_01x08, J6 Conn_01x04, J7 Conn_01x08, J8 Conn_01x06, J9 Conn_01x08

Commit message: route primary functional traces
Parts:
- added J10: Conn_01x04, Connector_PinHeader_2.54mm:PinHeader_1x04_P2.54mm_Vertical, F.Cu at (181.0, 130.9)
- added J11: Conn_01x06, Connector_PinHeader_2.54mm:PinHeader_1x06_P2.54mm_Vertical, F.Cu at (163.4, 130.9)
- added J12: Conn_01x08, Connector_PinHeader_2.54mm:PinHeader_1x08_P2.54mm_Vertical, F.Cu at (140.6, 127.3)
- added J13: Conn_01x08, Connector_PinHeader_2.54mm:PinHeader_1x08_P2.54mm_Vertical, F.Cu at (97.1, 127.3)
- added J14: Conn_01x08, Connector_PinHeader_2.54mm:PinHeader_1x08_P2.54mm_Vertical, F.Cu at (140.6, 130.9)
- added J15: Conn_01x08, Connector_PinHeader_2.54mm:PinHeader_1x08_P2.54mm_Vertical, F.Cu at (169.0, 127.3)
- added J16: Conn_01x16, Connector_PinHeader_2.54mm:PinHeader_1x16_P2.54mm_Vertical, F.Cu at (135.2, 130.9)
Connections:
- M1 pad 1: unconnected-(M1-A0-Pad1) -> /A0
- M1 pad 10: unconnected-(M1-A9-Pad10) -> /A9
- M1 pad 11: unconnected-(M1-A10-Pad11) -> /A10
- M1 pad 12: unconnected-(M1-A11-Pad12) -> /A11
- M1 pad 13: unconnected-(M1-A12-Pad13) -> /A12
- M1 pad 14: unconnected-(M1-A13-Pad14) -> /A13
- M1 pad 15: unconnected-(M1-A14-Pad15) -> /A14
- M1 pad 16: unconnected-(M1-A15-Pad16) -> /A15
- M1 pad 17: unconnected-(M1-S0-Pad17) -> DEV0
- M1 pad 18: unconnected-(M1-S1-Pad18) -> DEV1
- M1 pad 19: unconnected-(M1-S2-Pad19) -> DEV2
- M1 pad 2: unconnected-(M1-A1-Pad2) -> /A1
- M1 pad 20: unconnected-(M1-S3-Pad20) -> DEV3
- M1 pad 21: unconnected-(M1-S4-Pad21) -> DEV4
- M1 pad 22: unconnected-(M1-S5-Pad22) -> DEV5
- M1 pad 23: unconnected-(M1-S6-Pad23) -> DEV6
- M1 pad 24: unconnected-(M1-S7-Pad24) -> DEV7
- M1 pad 25: unconnected-(M1-D0-Pad25) -> /D0
- M1 pad 26: unconnected-(M1-D1-Pad26) -> /D1
- M1 pad 27: unconnected-(M1-D2-Pad27) -> /D2
- M1 pad 28: unconnected-(M1-D3-Pad28) -> /D3
- M1 pad 29: unconnected-(M1-D4-Pad29) -> /D4
- M1 pad 3: unconnected-(M1-A2-Pad3) -> /A2
- M1 pad 30: unconnected-(M1-D5-Pad30) -> /D5
- M1 pad 31: unconnected-(M1-D6-Pad31) -> /D6
- M1 pad 32: unconnected-(M1-D7-Pad32) -> /D7
- M1 pad 33: unconnected-(M1-E-Pad33) -> E
- M1 pad 34: unconnected-(M1-~{RESET}-Pad34) -> ~{RESET}
- M1 pad 35: unconnected-(M1-R/~{W}-Pad35) -> R/~{W}
- M1 pad 36: unconnected-(M1-Q-Pad36) -> Q
- M1 pad 37: unconnected-(M1-VCC-Pad37) -> +5V
- M1 pad 38: unconnected-(M1-VSS-Pad38) -> GND
- M1 pad 4: unconnected-(M1-A3-Pad4) -> /A3
- M1 pad 5: unconnected-(M1-A4-Pad5) -> /A4
- M1 pad 6: unconnected-(M1-A5-Pad6) -> /A5
- M1 pad 7: unconnected-(M1-A6-Pad7) -> /A6
- M1 pad 8: unconnected-(M1-A7-Pad8) -> /A7
- M1 pad 9: unconnected-(M1-A8-Pad9) -> /A8
- M2 pad 1: unconnected-(M2-A0-Pad1) -> /A0
- M2 pad 10: unconnected-(M2-A9-Pad10) -> /A9
- M2 pad 11: unconnected-(M2-A10-Pad11) -> /A10
- M2 pad 12: unconnected-(M2-A11-Pad12) -> /A11
- M2 pad 13: unconnected-(M2-A12-Pad13) -> /A12
- M2 pad 14: unconnected-(M2-A13-Pad14) -> /A13
- M2 pad 15: unconnected-(M2-A14-Pad15) -> /A14
- M2 pad 16: unconnected-(M2-A15-Pad16) -> /A15
- M2 pad 17: unconnected-(M2-S0-Pad17) -> DEV0
- M2 pad 18: unconnected-(M2-S1-Pad18) -> DEV1
- M2 pad 19: unconnected-(M2-S2-Pad19) -> DEV2
- M2 pad 2: unconnected-(M2-A1-Pad2) -> /A1
- M2 pad 20: unconnected-(M2-S3-Pad20) -> DEV3
- M2 pad 21: unconnected-(M2-S4-Pad21) -> DEV4
- M2 pad 22: unconnected-(M2-S5-Pad22) -> DEV5
- M2 pad 23: unconnected-(M2-S6-Pad23) -> DEV6
- M2 pad 24: unconnected-(M2-S7-Pad24) -> DEV7
- M2 pad 25: unconnected-(M2-D0-Pad25) -> /D0
- M2 pad 26: unconnected-(M2-D1-Pad26) -> /D1
- M2 pad 27: unconnected-(M2-D2-Pad27) -> /D2
- M2 pad 28: unconnected-(M2-D3-Pad28) -> /D3
- M2 pad 29: unconnected-(M2-D4-Pad29) -> /D4
- M2 pad 3: unconnected-(M2-A2-Pad3) -> /A2
- M2 pad 30: unconnected-(M2-D5-Pad30) -> /D5
- M2 pad 31: unconnected-(M2-D6-Pad31) -> /D6
- M2 pad 32: unconnected-(M2-D7-Pad32) -> /D7
- M2 pad 33: unconnected-(M2-E-Pad33) -> E
- M2 pad 34: unconnected-(M2-~{RESET}-Pad34) -> ~{RESET}
- M2 pad 35: unconnected-(M2-R/~{W}-Pad35) -> R/~{W}
- M2 pad 36: unconnected-(M2-Q-Pad36) -> Q
- M2 pad 37: unconnected-(M2-VCC-Pad37) -> +5V
- M2 pad 38: unconnected-(M2-VSS-Pad38) -> GND
- M2 pad 4: unconnected-(M2-A3-Pad4) -> /A3
- M2 pad 5: unconnected-(M2-A4-Pad5) -> /A4
- M2 pad 6: unconnected-(M2-A5-Pad6) -> /A5
- M2 pad 7: unconnected-(M2-A6-Pad7) -> /A6
- M2 pad 8: unconnected-(M2-A7-Pad8) -> /A7
- M2 pad 9: unconnected-(M2-A8-Pad9) -> /A8
- M3 pad 1: unconnected-(M3-A0-Pad1) -> /A0
- M3 pad 10: unconnected-(M3-A9-Pad10) -> /A9
- M3 pad 11: unconnected-(M3-A10-Pad11) -> /A10
- M3 pad 12: unconnected-(M3-A11-Pad12) -> /A11
- M3 pad 13: unconnected-(M3-A12-Pad13) -> /A12
- M3 pad 14: unconnected-(M3-A13-Pad14) -> /A13
- M3 pad 15: unconnected-(M3-A14-Pad15) -> /A14
- M3 pad 16: unconnected-(M3-A15-Pad16) -> /A15
- M3 pad 17: unconnected-(M3-S0-Pad17) -> DEV0
- M3 pad 18: unconnected-(M3-S1-Pad18) -> DEV1
- M3 pad 19: unconnected-(M3-S2-Pad19) -> DEV2
- M3 pad 2: unconnected-(M3-A1-Pad2) -> /A1
- M3 pad 20: unconnected-(M3-S3-Pad20) -> DEV3
- M3 pad 21: unconnected-(M3-S4-Pad21) -> DEV4
- M3 pad 22: unconnected-(M3-S5-Pad22) -> DEV5
- M3 pad 23: unconnected-(M3-S6-Pad23) -> DEV6
- M3 pad 24: unconnected-(M3-S7-Pad24) -> DEV7
- M3 pad 25: unconnected-(M3-D0-Pad25) -> /D0
- M3 pad 26: unconnected-(M3-D1-Pad26) -> /D1
- M3 pad 27: unconnected-(M3-D2-Pad27) -> /D2
- M3 pad 28: unconnected-(M3-D3-Pad28) -> /D3
- M3 pad 29: unconnected-(M3-D4-Pad29) -> /D4
- M3 pad 3: unconnected-(M3-A2-Pad3) -> /A2
- M3 pad 30: unconnected-(M3-D5-Pad30) -> /D5
- M3 pad 31: unconnected-(M3-D6-Pad31) -> /D6
- M3 pad 32: unconnected-(M3-D7-Pad32) -> /D7
- M3 pad 33: unconnected-(M3-E-Pad33) -> E
- M3 pad 34: unconnected-(M3-~{RESET}-Pad34) -> ~{RESET}
- M3 pad 35: unconnected-(M3-R/~{W}-Pad35) -> R/~{W}
- M3 pad 36: unconnected-(M3-Q-Pad36) -> Q
- M3 pad 37: unconnected-(M3-VCC-Pad37) -> +5V
- M3 pad 38: unconnected-(M3-VSS-Pad38) -> GND
- M3 pad 4: unconnected-(M3-A3-Pad4) -> /A3
- M3 pad 5: unconnected-(M3-A4-Pad5) -> /A4
- M3 pad 6: unconnected-(M3-A5-Pad6) -> /A5
- M3 pad 7: unconnected-(M3-A6-Pad7) -> /A6
- M3 pad 8: unconnected-(M3-A7-Pad8) -> /A7
- M3 pad 9: unconnected-(M3-A8-Pad9) -> /A8
- M4 pad 1: unconnected-(M4-A0-Pad1) -> /A0
- M4 pad 10: unconnected-(M4-A9-Pad10) -> /A9
- M4 pad 11: unconnected-(M4-A10-Pad11) -> /A10
- M4 pad 12: unconnected-(M4-A11-Pad12) -> /A11
- M4 pad 13: unconnected-(M4-A12-Pad13) -> /A12
- M4 pad 14: unconnected-(M4-A13-Pad14) -> /A13
- M4 pad 15: unconnected-(M4-A14-Pad15) -> /A14
- M4 pad 16: unconnected-(M4-A15-Pad16) -> /A15
- M4 pad 17: unconnected-(M4-S0-Pad17) -> DEV0
- M4 pad 18: unconnected-(M4-S1-Pad18) -> DEV1
- M4 pad 19: unconnected-(M4-S2-Pad19) -> DEV2
- M4 pad 2: unconnected-(M4-A1-Pad2) -> /A1
- M4 pad 20: unconnected-(M4-S3-Pad20) -> DEV3
- M4 pad 21: unconnected-(M4-S4-Pad21) -> DEV4
- M4 pad 22: unconnected-(M4-S5-Pad22) -> DEV5
- M4 pad 23: unconnected-(M4-S6-Pad23) -> DEV6
- M4 pad 24: unconnected-(M4-S7-Pad24) -> DEV7
- M4 pad 25: unconnected-(M4-D0-Pad25) -> /D0
- M4 pad 26: unconnected-(M4-D1-Pad26) -> /D1
- M4 pad 27: unconnected-(M4-D2-Pad27) -> /D2
- M4 pad 28: unconnected-(M4-D3-Pad28) -> /D3
- M4 pad 29: unconnected-(M4-D4-Pad29) -> /D4
- M4 pad 3: unconnected-(M4-A2-Pad3) -> /A2
- M4 pad 30: unconnected-(M4-D5-Pad30) -> /D5
- M4 pad 31: unconnected-(M4-D6-Pad31) -> /D6
- M4 pad 32: unconnected-(M4-D7-Pad32) -> /D7
- M4 pad 33: unconnected-(M4-E-Pad33) -> E
- M4 pad 34: unconnected-(M4-~{RESET}-Pad34) -> ~{RESET}
- M4 pad 35: unconnected-(M4-R/~{W}-Pad35) -> R/~{W}
- M4 pad 36: unconnected-(M4-Q-Pad36) -> Q
- M4 pad 37: unconnected-(M4-VCC-Pad37) -> +5V
- M4 pad 38: unconnected-(M4-VSS-Pad38) -> GND
- M4 pad 4: unconnected-(M4-A3-Pad4) -> /A3
- M4 pad 5: unconnected-(M4-A4-Pad5) -> /A4
- M4 pad 6: unconnected-(M4-A5-Pad6) -> /A5
- M4 pad 7: unconnected-(M4-A6-Pad7) -> /A6
- M4 pad 8: unconnected-(M4-A7-Pad8) -> /A7
- M4 pad 9: unconnected-(M4-A8-Pad9) -> /A8
Routing:
- net ~{RESET}: track 0.00 -> 361.9 mm, vias 0 -> 7
- net R/~{W}: track 0.00 -> 357.0 mm, vias 0 -> 7
- net +5V: track 0.00 -> 231.1 mm
- net /D0: track 0.00 -> 223.4 mm, vias 0 -> 4
- net /D1: track 0.00 -> 218.5 mm, vias 0 -> 4
- net E: track 0.00 -> 214.6 mm, vias 0 -> 4
- net /D2: track 0.00 -> 214.5 mm, vias 0 -> 4
- net /D3: track 0.00 -> 206.7 mm, vias 0 -> 4
- net /D7: track 0.00 -> 205.7 mm, vias 0 -> 3
- net /D4: track 0.00 -> 201.4 mm, vias 0 -> 4
- net /D6: track 0.00 -> 199.4 mm, vias 0 -> 4
- net Q: track 0.00 -> 197.3 mm, vias 0 -> 3
- net /D5: track 0.00 -> 194.5 mm, vias 0 -> 2
- net DEV7: track 0.00 -> 192.8 mm, vias 0 -> 2
- net DEV5: track 0.00 -> 192.1 mm, vias 0 -> 2
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- added copper zone on B.Cu, net GND
- added copper zone on F.Cu, net GND

Commit message: finish routing
Parts:
- removed J11: Conn_01x06, Connector_PinHeader_2.54mm:PinHeader_1x06_P2.54mm_Vertical
Connections:
- J13 pad 7: ~{Q} -> unconnected-(J13-Pin_7-Pad7)
- J13 pad 8: ~{E} -> unconnected-(J13-Pin_8-Pad8)
Routing:
- net ~{NMI}: track 0.00 -> 119.6 mm, vias 0 -> 5
- net ~{IRQ}: track 0.00 -> 118.8 mm, vias 0 -> 5
- net ~{FIRQ}: track 0.00 -> 117.3 mm, vias 0 -> 5
- net /D5: track 194.5 -> 193.4 mm
- net /D3: track 206.7 -> 205.6 mm
- net /D4: track 201.4 -> 200.3 mm
- net /D1: track 218.5 -> 217.4 mm
- net /D0: track 223.4 -> 222.4 mm
- net /D2: track 214.5 -> 213.5 mm
- net /D6: track 199.4 -> 198.4 mm
- net R/~{W}: track 357.0 -> 356.3 mm, vias 7 -> 6
- net /A7: track 184.0 -> 184.7 mm
- net ~{RESET}: track 361.9 -> 361.8 mm, vias 7 -> 6
- net GND: vias 0 -> 61
